Commit message: added a fullcollision model and replaced all collision meshes with primitives

File: mujoco_playground/_src/locomotion/bez2/xmls/meshes/robot22.urdf (robot description, URDF)
Before this commit: robot bez2, 23 links, 22 joints
Links:
- link trunk: geometry collision box size=0.18229 0.17215 0.16665; visual mesh filename=base_link.stl scale=0.001 0.001 0.001
